File: power/power.sch (KiCad schematic (older format))
At the start: 90 parts, among them J1 Conn_01x02_Female, J2 Conn_01x02_Female, J3 CONN_02X03, J4 Conn_01x06_Female, Q1 BS170, Q10 BS170, Q11 BS170, Q12 BSB014N04LX3, Q2 BS170, Q3 BS170, Q4 BS170, Q5 BS170, Q6 BS170, Q7 BS170, Q8 BS170, Q9 BS170, U1 MAX1648, U2 TPS2592xx, U3 LMC6482

Commit message: complete schematic
Parts:
- removed C1, C12, C13, C14, C16, C5, C6, C7, C?: C, Capacitor_SMD:C_0805_2012Metric_Pad1.15x1.40mm_HandSolder, symbol Device:C
- removed C17: CP1, Capacitor_SMD:C_0805_2012Metric_Pad1.15x1.40mm_HandSolder, symbol Device:CP1
- removed D7: LED, LED_SMD:LED_0805_2012Metric_Pad1.15x1.40mm_HandSolder, symbol Device:LED
- removed Q10, Q4, Q8, Q9: BS170, Package_TO_SOT_THT:TO-92_Inline, symbol Transistor_FET:BS170
- removed R12, R14, R20, R21, R23, R24, R25, R28, R?: R, Resistor_SMD:R_0805_2012Metric_Pad1.15x1.40mm_HandSolder, symbol Device:R
- removed R16, R7: 100, Resistor_SMD:R_0805_2012Metric_Pad1.15x1.40mm_HandSolder, symbol Device:R
- removed TH5, TH6, TH7: Thermistor, footprints:Thermistor, symbol Device:Thermistor
- removed U3: LMC6482, footprints:SOIC127P600X175-8N, symbol Amplifier_Operational:LMC6482
- removed U?: APE1707M-12-HF, Package_SO:SOIC-8_3.9x4.9mm_P1.27mm, symbol Regulator_Switching:APE1707M-12-HF
- removed U?: APE1707M-50-HF, Package_SO:SOIC-8_3.9x4.9mm_P1.27mm, symbol Regulator_Switching:APE1707M-50-HF
- added C?: 0.1uF, Capacitor_SMD:C_0805_2012Metric_Pad1.15x1.40mm_HandSolder, symbol Device:CP1
- added C?: 1uF, Capacitor_SMD:C_0805_2012Metric_Pad1.15x1.40mm_HandSolder, symbol Device:CP1
- added J? (x5): Conn_01x02_Female, Connector_PinHeader_1.00mm:PinHeader_1x02_P1.00mm_Vertical, symbol Connector:Conn_01x02_Female
- added R? (x5): 1.5K, Resistor_SMD:R_0805_2012Metric_Pad1.15x1.40mm_HandSolder, symbol Device:R
- added SW?: SW_Push, symbol Switch:SW_Push
- added TH? (x3): Thermistor, footprints:Thermistor, symbol Device:Thermistor
- D?: value D_Zener -> 12.5V
- R11: value R -> 1.5K
- R26: value R -> 133
- R27: value R -> 20
- R29: value R -> 115K
Connections:
- net +5V is gone; now on net +12V: C?.2, U?.1 (IN)
- net B3- is gone; now on net GND: J4.3 (Pin_3), R10.2
- net B4+ is gone; now on net B1B+: D2.1 (K), D?.1 (K), J?.4 (Pin_4), R26.1, U2.3 (VIN), U2.4 (VIN), U2.5 (VIN)
- net B6- is gone; now on net GND: J4.6 (Pin_6), R19.2
- net +12V: now also C?.1
- net +3V3: now also J?.1 (Pin_1), J?.1 (Pin_1), J?.1 (Pin_1), J?.1 (Pin_1), J?.1 (Pin_1)
- net BAT+: now also SW?.1; no longer D1.2 (A)
- net GND: now also R11.2, U2.1 (dV/dT), C?.2, J?.2 (Pin_2), J?.2 (Pin_2), J?.2 (Pin_2), J?.2 (Pin_2), J?.2 (Pin_2), R?.2, R?.2, R?.2, R?.2, R?.2; no longer TH1.2, TH2.2, TH3.2
- net B1A+: now reaches Q1.1 (D)
- net B1A+: now also D1.1 (K), D2.2 (A), J?.1 (Pin_1), TH1.1
- net B1B+: now reaches Q5.1 (D)
- net B1B+: now also C?.1, TH?.1
- net +12.5V: no longer names the net of U2.6 (OUT), U2.7 (OUT), U2.8 (OUT)
- net +12.5V: now also C?.2
- removed net B1+: D1.1 (K), D2.2 (A), J?.1 (Pin_1), R11.1
- net B1- renamed B1A-
- net B1A-: now also TH2.1
- net B2- renamed B2A-
- net B2A-: now also TH3.1
- net B4- renamed B1B-
- net B1B-: now also TH?.1
- net B5- renamed B2B-
- net B2B-: now also TH?.1
- net FET1 renamed FET1A
- net FET2 renamed FET2A
- net FET3 renamed FET3A
- net FET4 renamed FET1B
- net FET5 renamed FET2B
- net FET6 renamed FET3B
- removed net T1: R11.2, TH1.1, U?.14 ((PCINT22/ADC3/INT0/ACMPN2)PD6)
- net T2 renamed V2A
- net V2A: now also TH2.2, R?.1; no longer TH2.1
- net T3 renamed V3A
- net V3A: now also TH3.2, R?.1; no longer TH3.1
- net T4 renamed V1B
- net V1B: now also R?.1, TH?.2
- net T5 renamed V2B
- net V2B: now also R?.1, TH?.2
- net T6 renamed V3B
- net V3B: now also R?.1, TH?.2
- new net: D1.2 (A), SW?.2
- new net V1A: R11.1, TH1.2, U?.14 ((PCINT22/ADC3/INT0/ACMPN2)PD6)
Other:
- note added: "0V\n"
- note added: "12.3V"
- note added: "12.3V \n4A\n----->"
- note added: "1K Ohms"
- note added: "4.1V"
- note added: "8.2V"
- note added: "Connections"
- note added: "LDO\n12.3V -> 3.3V"
- note added: "Power INPUT Connectors"
- note added: "To Baro1"
- note added: "To Baro2"
- note added: "To GPS"
- note added: "To IMU"
- note added: "To Radio"
- note added: "To Recovery (12.3, 4A)"
- note added: "To Teensy"
- note added: "Variable Output 12.3V"
- note added: "Voltage Monitoring\n"
- note removed: "12.5V \n2A\n----->"
- note removed: "Buck\n12.5V -> 12V"
- note removed: "Buck\n12V -> 5V"
- note removed: "CC Discharging - 2000 mA"
- note removed: "LDO\n5V -> 3.3V"
- note removed: "Need to duplicate for each sensor"
- note removed: "Power Connectors"
- note removed: "To Recovery"
- note removed: "To Sensors and Teensy"
- moved on the sheet: C10, C11, C2, C3, C4, C8, C9, C?, D1, D2, D3, D4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
